File: Human_Tracker.kicad_sch (KiCad schematic)
At the start: 59 parts, among them U1 TPS54233QDRQ1, U2 ICS-43434_C5656610, U3 ICS-43434_C5656610, U4 ADM7172ACPZ-3.3-R7, U5 BME680, U6 ESP32-S3-WROOM-1(N16R8), U7 MLX90640ESF-BAB-000-TU, U8 FRC0805F1400TS 140

Commit message: Commit
Parts:
- C1, C12, C13, C2, C3, C5, C6: footprint PCM_JLCPCB:C_0805 -> lcsc_footprints:C1712_C0805
- C10, C15, C16, C17, C18, C4: footprint Capacitor_SMD:C_0805_2012Metric -> lcsc_footprints:C1712_C0805
- C11: footprint lcsc_footprints:C1791_C0805 -> lcsc_footprints:C1712_C0805
- C7: footprint lcsc_footprints:C124129_C0805 -> lcsc_footprints:C1712_C0805
- C8: footprint lcsc_footprints:C29277_C0805 -> lcsc_footprints:C1712_C0805
- C9: footprint lcsc_footprints:C49678_C0805 -> lcsc_footprints:C1712_C0805
- R1, R2, R6: footprint PCM_JLCPCB:R_0805 -> lcsc_footprints:C17414_R0805
- R10, R9: footprint lcsc_footprints:C17561_R0805 -> lcsc_footprints:C17414_R0805
- R12: footprint lcsc_footprints:C25611_R0805 -> lcsc_footprints:C17414_R0805
- R13, R14, R15, R16, R8: footprint Resistor_SMD:R_0805_2012Metric -> lcsc_footprints:C17414_R0805
- R3, R5: footprint lcsc_footprints:C26023_R0805 -> lcsc_footprints:C17414_R0805
- R4: footprint lcsc_footprints:C2933366_R0805 -> lcsc_footprints:C17414_R0805
- R7: footprint lcsc_footprints:C17534_R0805 -> lcsc_footprints:C17414_R0805
Changed lines of the file:
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@@
 			)
 		)
-		(property "Footprint" "Resistor_SMD:R_0805_2012Metric"
+		(property "Footprint" "lcsc_footprints:C17414_R0805"
 			(at 450.342 101.6 90)
 			(hide yes)
@@
 			)
 		)
-		(property "Footprint" "Resistor_SMD:R_0805_2012Metric"
+		(property "Footprint" "lcsc_footprints:C17414_R0805"
 			(at 436.372 97.79 90)
 			(hide yes)
@@
 			)
 		)
-		(property "Footprint" "PCM_JLCPCB:C_0805"
+		(property "Footprint" "lcsc_footprints:C1712_C0805"
 			(at 196.342 278.13 90)
 			(hide yes)
@@
 			)
 		)
-		(property "Footprint" "Resistor_SMD:R_0805_2012Metric"
+		(property "Footprint" "lcsc_footprints:C17414_R0805"
 			(at 174.752 115.57 90)
 			(hide yes)
@@
 			)
 		)
-		(property "Footprint" "Resistor_SMD:R_0805_2012Metric"
+		(property "Footprint" "lcsc_footprints:C17414_R0805"
 			(at 337.312 113.03 90)
 			(hide yes)
@@
 			)
 		)
-		(property "Footprint" "Capacitor_SMD:C_0805_2012Metric"
+		(property "Footprint" "lcsc_footprints:C1712_C0805"
 			(at 402.2852 92.71 0)
 			(hide yes)
@@
 			)
 		)
-		(property "Footprint" "Capacitor_SMD:C_0805_2012Metric"
+		(property "Footprint" "lcsc_footprints:C1712_C0805"
 			(at 390.8552 92.71 0)
 			(hide yes)
@@
 			)
 		)
-		(property "Footprint" "lcsc_footprints:C29277_C0805"
+		(property "Footprint" "lcsc_footprints:C1712_C0805"
 			(at 265.1252 166.37 0)
 			(hide yes)
@@
 			)
 		)
-		(property "Footprint" "PCM_JLCPCB:C_0805"
+		(property "Footprint" "lcsc_footprints:C1712_C0805"
 			(at 135.382 313.69 90)
 			(hide yes)
@@
 			)
 		)
-		(property "Footprint" "lcsc_footprints:C17534_R0805"
+		(property "Footprint" "lcsc_footprints:C17414_R0805"
 			(at 162.56 302.26 0)
 			(hide yes)
@@
 			)
 		)
-		(property "Footprint" "Capacitor_SMD:C_0805_2012Metric"
+		(property "Footprint" "lcsc_footprints:C1712_C0805"
 			(at 266.3952 116.84 0)
 			(hide yes)
@@
 			)
 		)
-		(property "Footprint" "lcsc_footprints:C1791_C0805"
+		(property "Footprint" "lcsc_footprints:C1712_C0805"
 			(at 194.31 299.72 0)
 			(hide yes)
@@
 			)
 		)
-		(property "Footprint" "PCM_JLCPCB:R_0805"
+		(property "Footprint" "lcsc_footprints:C17414_R0805"
 			(at 89.662 297.18 90)
 			(hide yes)
@@
 			)
 		)
-		(property "Footprint" "PCM_JLCPCB:C_0805"
+		(property "Footprint" "lcsc_footprints:C1712_C0805"
 			(at 123.952 317.5 90)
 			(hide yes)
@@
 			)
 		)
-		(property "Footprint" "lcsc_footprints:C49678_C0805"
+		(property "Footprint" "lcsc_footprints:C1712_C0805"
 			(at 275.2852 166.37 0)
 			(hide yes)
@@
 			)
 		)
-		(property "Footprint" "Capacitor_SMD:C_0805_2012Metric"
+		(property "Footprint" "lcsc_footprints:C1712_C0805"
 			(at 103.8352 95.25 0)
 			(hide yes)
@@
 			)
 		)
-		(property "Footprint" "PCM_JLCPCB:R_0805"
+		(property "Footprint" "lcsc_footprints:C17414_R0805"
 			(at 150.622 290.83 90)
 			(hide yes)
@@
 			)
 		)
-		(property "Footprint" "lcsc_footprints:C17561_R0805"
+		(property "Footprint" "lcsc_footprints:C17414_R0805"
 			(at 266.7 221.488 90)
 			(hide yes)
@@
 			)
 		)
-		(property "Footprint" "lcsc_footprints:C26023_R0805"
+		(property "Footprint" "lcsc_footprints:C17414_R0805"
 			(at 143.002 185.42 90)
 			(hide yes)
@@
 			)
 		)
-		(property "Footprint" "lcsc_footprints:C26023_R0805"
+		(property "Footprint" "lcsc_footprints:C17414_R0805"
 			(at 98.552 185.42 90)
 			(hide yes)
@@
 			)
 		)
-		(property "Footprint" "PCM_JLCPCB:C_0805"
+		(property "Footprint" "lcsc_footprints:C1712_C0805"
 			(at 231.902 278.13 90)
 			(hide yes)
@@
 			)
 		)
-		(property "Footprint" "PCM_JLCPCB:C_0805"
+		(property "Footprint" "lcsc_footprints:C1712_C0805"
 			(at 97.282 303.53 90)
 			(hide yes)
@@
 			)
 		)
-		(property "Footprint" "PCM_JLCPCB:C_0805"
+		(property "Footprint" "lcsc_footprints:C1712_C0805"
 			(at 93.472 283.21 90)
 			(hide yes)
@@
 			)
 		)
-		(property "Footprint" "lcsc_footprints:C124129_C0805"
+		(property "Footprint" "lcsc_footprints:C1712_C0805"
 			(at 142.24 293.37 0)
 			(hide yes)
@@
 			)
 		)
-		(property "Footprint" "lcsc_footprints:C17561_R0805"
+		(property "Footprint" "lcsc_footprints:C17414_R0805"
 			(at 256.54 224.028 90)
 			(hide yes)
@@
 			)
 		)
-		(property "Footprint" "lcsc_footprints:C2933366_R0805"
+		(property "Footprint" "lcsc_footprints:C17414_R0805"
 			(at 147.32 323.85 0)
 			(hide yes)
@@
 			)
 		)
-		(property "Footprint" "Capacitor_SMD:C_0805_2012Metric"
+		(property "Footprint" "lcsc_footprints:C1712_C0805"
 			(at 279.0952 116.84 0)
 			(hide yes)
@@
 			)
 		)
-		(property "Footprint" "PCM_JLCPCB:C_0805"
+		(property "Footprint" "lcsc_footprints:C1712_C0805"
 			(at 82.042 294.64 90)
 			(hide yes)
@@
 			)
 		)
-		(property "Footprint" "PCM_JLCPCB:R_0805"
+		(property "Footprint" "lcsc_footprints:C17414_R0805"
 			(at 89.662 307.34 90)
 			(hide yes)
@@
 			)
 		)
-		(property "Footprint" "Resistor_SMD:R_0805_2012Metric"
+		(property "Footprint" "lcsc_footprints:C17414_R0805"
 			(at 354.838 110.49 90)
 			(hide yes)
@@
 			)
 		)
-		(property "Footprint" "Capacitor_SMD:C_0805_2012Metric"
+		(property "Footprint" "lcsc_footprints:C1712_C0805"
 			(at 195.2752 95.25 0)
 			(hide yes)
@@
 			)
 		)
-		(property "Footprint" "lcsc_footprints:C25611_R0805"
+		(property "Footprint" "lcsc_footprints:C17414_R0805"
 			(at 308.102 267.97 90)
 			(hide yes)
