File: Human_Tracker.kicad_pcb (KiCad board)
At the start: 2 copper layers, 49 parts, among them U1 TPS54233QDRQ1, U2 ICS-43434_C5656610, U3 ICS-43434_C5656610, U4 ADM7172ACPZ-3.3-R7, U5 BME680, U6 ESP32-S3-WROOM-1(N16R8), U7 MLX90640ESF-BAB-000-TU, U8 FRC0805F1400TS 140

Commit message: Commit
Parts:
- added C1: 10uF, lcsc_footprints:C1712_C0805, F.Cu at (105.7, 140.5)
- added C12: 4.7uF, lcsc_footprints:C1712_C0805, F.Cu at (115.3, 139.5)
- added C13: 4.7uF, lcsc_footprints:C1712_C0805, F.Cu at (115.7, 129.9)
- added C2: 100nF, lcsc_footprints:C1712_C0805, F.Cu at (103.6, 140.5)
- added C3: 10nF, lcsc_footprints:C1712_C0805, F.Cu at (111.8, 140.5)
- added C5: 47pF, lcsc_footprints:C1712_C0805, F.Cu at (108.2, 128.5)
- added C6: 4.7nF, lcsc_footprints:C1712_C0805, F.Cu at (104.2, 128.6)
- added R1: 150kΩ, lcsc_footprints:C17414_R0805, F.Cu at (108.6, 139.4)
- added R2: 62kΩ, lcsc_footprints:C17414_R0805, F.Cu at (108.6, 141.6)
- added R6: 10kΩ, lcsc_footprints:C17414_R0805, F.Cu at (96.8, 133.4)
- C10, C15, C16, C17, C18, C4: footprint Capacitor_SMD:C_0805_2012Metric -> lcsc_footprints:C1712_C0805
- C11: footprint lcsc_footprints:C1791_C0805 -> lcsc_footprints:C1712_C0805
- C7: footprint lcsc_footprints:C124129_C0805 -> lcsc_footprints:C1712_C0805
- C8: footprint lcsc_footprints:C29277_C0805 -> lcsc_footprints:C1712_C0805
- C9: footprint lcsc_footprints:C49678_C0805 -> lcsc_footprints:C1712_C0805
- R10, R9: footprint lcsc_footprints:C17561_R0805 -> lcsc_footprints:C17414_R0805
- R12: footprint lcsc_footprints:C25611_R0805 -> lcsc_footprints:C17414_R0805
- R13, R14, R15, R16, R8: footprint Resistor_SMD:R_0805_2012Metric -> lcsc_footprints:C17414_R0805
- R3, R5: footprint lcsc_footprints:C26023_R0805 -> lcsc_footprints:C17414_R0805
- R4: footprint lcsc_footprints:C2933366_R0805 -> lcsc_footprints:C17414_R0805
- R7: footprint lcsc_footprints:C17534_R0805 -> lcsc_footprints:C17414_R0805
- moved U3 131.0 mm to (257.9, 118.1)
- moved C10 116.4 mm to (258.0, 114.8)
- moved R12 104.3 mm to (225.3, 127.7), turned to 90 degrees
- moved H3 98.8 mm to (243.8, 116.3), turned to 90 degrees
- moved U6 97.7 mm to (221.5, 112.3)
- moved R13 93.3 mm to (82.0, 122.8), turned to -90 degrees
- moved SM1 90.8 mm to (85.3, 109.3), turned to 180 degrees
- moved R14 89.2 mm to (85.7, 123.8)
- moved R8 88.2 mm to (258.0, 121.4)
- moved R11 83.6 mm to (205.9, 103.0)
- moved R9 76.8 mm to (192.5, 132.8), turned to 180 degrees
- moved H4 75.6 mm to (221.5, 132.8)
- moved C4 75.1 mm to (69.5, 116.8)
- moved R10 74.7 mm to (192.5, 130.2), turned to 180 degrees
- moved H2 67.5 mm to (199.6, 116.3), turned to -90 degrees
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Other:
- board outline added: 200 x 50 mm
- copper layers 2 -> 4

Commit message: petite correction
Parts:
- C17: value 10µ -> 10uF; footprint lcsc_footprints:C1712_C0805 -> lcsc_footprints:C15850_C0805
- moved U6 6.36 mm to (221.0, 105.9)
- moved R11 2.10 mm to (204.5, 101.5)
- moved U5 1.12 mm to (86.0, 118.5), turned to 90 degrees
- moved C14 1.08 mm to (205.9, 98.5)
Connections:
- C17 pad 1: +3.3V -> GND
- C17 pad 2: GND -> +3.3V
