File: _autosave-Human_Tracker.kicad_sch (KiCad schematic)
At the start: 59 parts, among them U1 TPS54233QDRQ1, U2 ICS-43434_C5656610, U3 ICS-43434_C5656610, U4 ADM7172ACPZ-3.3-R7, U5 BME680, U6 ESP32-S3-WROOM-1(N16R8), U7 MLX90640ESF-BAB-000-TU, U8 FRC0805F1400TS 140

Commit message: petite correction
Parts:
- renumbered C19 to C17
Changed lines of the file:
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@@
 		(dnp no)
 		(fields_autoplaced yes)
-		(property "Reference" "C19"
+		(property "Reference" "C17"
 			(at 403.86 87.6299 90)
 			(show_name no)
@@
 			(project "Human_Tracker"
 				(path "/21992c97-7c29-4ade-9a85-42ee1fb0a3a3"
-					(reference "C19")
+					(reference "C17")
 					(unit 1)
 				)
